Commit message: All changes and final humble commit.

File: mushr_description/robots/mushr_nano.urdf.xacro (robot description, xacro)
@@ -107,8 +107,8 @@
 	<joint
 		name="base_link_to_laser_link"
-		type="fixed" >
+		type="fixed">
 		<origin
 			xyz="-0.035325 0 0.10775"
-			rpy="0 0 0" />
+			rpy="0 0 3.14159" />
 		<parent
 			link="base_link" />

File: mushr_description/robots/mushr_tx2.urdf.xacro (robot description, xacro)
@@ -13,5 +13,5 @@
 	<xacro:mushr_ydlidar />
 	<xacro:sensor_d435 parent="base_link" >
-  		<origin xyz="0.10075 0.0 0.099" rpy="0 0 0" />
+  		<origin xyz="0.10075 0.0 0.099" rpy="0 0 3.14159" />
 	</xacro:sensor_d435>
 	<link name="front_left/wheel_steer_link"/>
